File: bldc_driver.kicad_sch (KiCad schematic)
At the start: 8 parts, among them Q1 DI030N10PT-AQ, Q2 DI030N10PT-AQ, Q3 DI030N10PT-AQ, Q4 DI030N10PT-AQ, Q5 DI030N10PT-AQ, Q6 DI030N10PT-AQ, U1 STM32F318K8Ux, U2 DRV8311S

Commit message: started driver circuit
Parts:
- added C8: 100nF, Capacitor_SMD:C_0402_1005Metric, symbol Device:C
Other:
- moved on the sheet: U1, U2
Changed lines of the file:
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@@
 	(symbol
 		(lib_id "Multi-ESC:DRV8311S")
-		(at 194.31 62.23 0)
+		(at 194.31 67.31 0)
 		(unit 1)
 		(body_style 1)
@@
 		(fields_autoplaced yes)
 		(property "Reference" "U2"
-			(at 197.7233 39.37 0)
+			(at 197.7233 44.45 0)
 			(show_name no)
 			(do_not_autoplace no)
@@
 		)
 		(property "Value" "DRV8311S"
-			(at 197.7233 41.91 0)
+			(at 197.7233 46.99 0)
 			(show_name no)
 			(do_not_autoplace no)
@@
 		)
 		(property "Footprint" "Package_DFN_QFN:WQFN-32-1EP_5x5mm_P0.5mm_EP3.1x3.1mm"
+			(at 194.31 102.87 0)
+			(hide yes)
+			(show_name no)
+			(do_not_autoplace no)
+			(effects
+				(font
+					(size 1.27 1.27)
+				)
+			)
+		)
+		(property "Datasheet" "https://www.ti.com/general/docs/suppproductinfo.tsp?distId=10&gotoUrl=https%3A%2F%2Fwww.ti.com%2Flit%2Fgpn%2Fdrv8320"
+			(at 194.31 100.33 0)
+			(hide yes)
+			(show_name no)
+			(do_not_autoplace no)
+			(effects
+				(font
+					(size 1.27 1.27)
+				)
+			)
+		)
+		(property "Description" "Three-Phase PWM Motor Driver, 3-20V supply, 5A peak current, SPI interface, WQFN-24"
 			(at 194.31 97.79 0)
 			(hide yes)
@@
 			)
 		)
-		(property "Datasheet" "https://www.ti.com/general/docs/suppproductinfo.tsp?distId=10&gotoUrl=https%3A%2F%2Fwww.ti.com%2Flit%2Fgpn%2Fdrv8320"
-			(at 194.31 95.25 0)
-			(hide yes)
-			(show_name no)
-			(do_not_autoplace no)
-			(effects
-				(font
-					(size 1.27 1.27)
-				)
-			)
-		)
-		(property "Description" "Three-Phase PWM Motor Driver, 3-20V supply, 5A peak current, SPI interface, WQFN-24"
-			(at 194.31 92.71 0)
-			(hide yes)
-			(show_name no)
-			(do_not_autoplace no)
-			(effects
-				(font
-					(size 1.27 1.27)
-				)
-			)
-		)
 		(property private "KLC_S4.4_AVDD" "This is the output of the 3.3V internal regulator"
-			(at 194.31 100.33 0)
+			(at 194.31 105.41 0)
 			(hide yes)
 			(show_name yes)
@@
 	(symbol
 		(lib_id "MCU_ST_STM32F3:STM32F318K8Ux")
-		(at 114.3 67.31 0)
+		(at 114.3 72.39 0)
 		(unit 1)
 		(body_style 1)
@@
 		(fields_autoplaced yes)
 		(property "Reference" "U1"
-			(at 118.9833 92.71 0)
+			(at 118.9833 97.79 0)
 			(show_name no)
 			(do_not_autoplace no)
@@
 		)
 		(property "Value" "STM32F318K8Ux"
-			(at 118.9833 95.25 0)
+			(at 118.9833 100.33 0)
 			(show_name no)
 			(do_not_autoplace no)
@@
 		)
 		(property "Footprint" "Package_DFN_QFN:QFN-32-1EP_5x5mm_P0.5mm_EP3.45x3.45mm"
-			(at 101.6 90.17 0)
+			(at 101.6 95.25 0)
 			(hide yes)
 			(show_name no)
@@
 		)
 		(property "Datasheet" "https://www.st.com/resource/en/datasheet/stm32f318k8.pdf"
-			(at 114.3 67.31 0)
+			(at 114.3 72.39 0)
 			(hide yes)
 			(show_name no)
@@
 		)
 		(property "Description" "STMicroelectronics Arm Cortex-M4 MCU, 64KB flash, 16KB RAM, 72 MHz, 1.65-1.95V, 23 GPIO, UFQFPN32"
-			(at 114.3 67.31 0)
+			(at 114.3 72.39 0)
 			(hide yes)
 			(show_name no)
@@
 					(unit 1)
 				)
+			)
+		)
+	)
+	(symbol
+		(lib_id "Device:C")
+		(at 102.87 33.02 0)
+		(unit 1)
+		(body_style 1)
+		(exclude_from_sim no)
+		(in_bom yes)
+		(on_board yes)
+		(in_pos_files yes)
+		(dnp no)
+		(property "Reference" "C8"
+			(at 104.14 30.734 0)
+			(show_name no)
+			(do_not_autoplace no)
+			(effects
+				(font
+					(size 1.27 1.27)
+				)
+				(justify left)
+			)
+		)
+		(property "Value" "100nF"
+			(at 104.14 35.814 0)
+			(show_name no)
+			(do_not_autoplace no)
+			(effects
+				(font
+					(size 1.27 1.27)
+				)
+				(justify left)
+			)
+		)
+		(property "Footprint" "Capacitor_SMD:C_0402_1005Metric"
+			(at 103.8352 36.83 0)
+			(hide yes)
+			(show_name no)
+			(do_not_autoplace no)
+			(effects
+				(font
+					(size 1.27 1.27)
+				)
+			)
+		)
+		(property "Datasheet" ""
+			(at 102.87 33.02 0)
+			(hide yes)
+			(show_name no)
+			(do_not_autoplace no)
+			(effects
+				(font
+					(size 1.27 1.27)
+				)
+			)
+		)
+		(property "Description" "Unpolarized capacitor"
+			(at 102.87 33.02 0)
+			(hide yes)
+			(show_name no)
+			(do_not_autoplace no)
+			(effects
+				(font
+					(size 1.27 1.27)
+				)
+			)
+		)
+		(pin "1"
+		)
+		(pin "2"
+		)
+		(instances
+			(project "Multi-ESC"
+				(path "/332a84c1-656a-45ff-900c-4414e0318fba/b7298b97-ad7a-472d-b821-c393573fc3f1"
+					(reference "C8")
+					(unit 1)
+				)

Commit message: wired mcu circuit
Parts:
- added C10, C9: 100nF, Capacitor_SMD:C_0402_1005Metric, symbol Device:C
- added C11, C13, C14: 1uF, Capacitor_SMD:C_0402_1005Metric, symbol Device:C
- added C12: 10nF, Capacitor_SMD:C_0402_1005Metric, symbol Device:C
- added C15, C16: C, Capacitor_SMD:C_0402_1005Metric, symbol Device:C
- added U4: MIC5504-1.8YM5, Package_TO_SOT_SMD:SOT-23-5, symbol Regulator_Linear:MIC5504-1.8YM5
- added Y1: Crystal_GND24, Crystal:Crystal_SMD_3225-4Pin_3.2x2.5mm, symbol Device:Crystal_GND24
- C8: value 100nF -> 4.7uF
Connections:
- net MISO: now reaches U2.18 (SDO)
- net MISO: now also U1.27 (PB4)
- net MOSI: now reaches U2.19 (SDI)
- net MOSI: now also U1.28 (PB5)
- net SCLK: now reaches U2.20 (SCLK)
- net SCLK: now also U1.26 (PB3)
- net CS: now reaches U2.21 (~{SCS})
- net CS: now also U1.11 (PA4)
- net GNDA: now reaches U2.23 (AGND)
- net GNDA: now also U1.6 (VSSA)
- net INHA: now reaches U2.25 (INHA)
- net INHA: now also U1.21 (PA11)
- net INLA: now reaches U2.26 (INLA)
- net INLA: now also U1.20 (PA10)
- net INHB: now reaches U2.27 (INHB)
- net INHB: now also U1.19 (PA9)
- net INLB: now reaches U2.28 (INLB)
- net INLB: now also U1.18 (PA8)
- net INHC: now reaches U2.29 (INHC)
- net INHC: now also U1.9 (PA2)
- net INLC: now reaches U2.30 (INLC)
- net INLC: now also U1.10 (PA3)
- net GND: now reaches U2.31 (PGND), U2.33 (PGND)
- net GND: now also C8.2, U1.16 (VSS), U1.32 (VSS), U1.33 (VSS), C10.2, C11.2, C12.2, C13.2, C14.2, C15.2, C16.2, C9.2, U4.2 (GND), Y1.2 (G), Y1.4 (G)
- net +1.8V: now reaches U1.1 (VDD)
- net +1.8V: now also C8.1, U1.17 (VDD), C10.1, C14.1, C9.1, U4.5 (VOUT)
- net IN_PWM: now reaches U1.12 (PA5)
- net BEMF_A: now reaches U1.13 (PA6)
- net BEMF_B: now reaches U1.14 (PA7)
- net BEMF_C: now reaches U1.15 (PB0)
- net HSE_IN: now reaches U1.2 (PF0)
- net HSE_IN: now also C15.1, Y1.1
- net SDA: now reaches U1.24 (PA14)
- net SCL: now reaches U1.25 (PA15)
- net HSE_OUT: now reaches U1.3 (PF1)
- net HSE_OUT: now also C16.1, Y1.3
- net +3.3V: now reaches U1.5 (VDDA)
- net +3.3V: now also C11.1, C12.1, C13.1, U4.1 (VIN)
- net VGND: now reaches U1.7 (PA0)
Other:
- moved on the sheet: C8
