File: bldc_driver.kicad_sch (KiCad schematic)
At the start: 58 parts, among them J1 Conn_01x01, J2 Conn_01x01, J3 Conn_01x01, Q1 DI030N10PT-AQ, Q2 DI030N10PT-AQ, Q3 DI030N10PT-AQ, Q4 DI030N10PT-AQ, Q5 DI030N10PT-AQ, Q6 DI030N10PT-AQ, Q7 Q_PMOS_DGS, U1 STM32F318K8Ux, U2 DRV8320SR, U4 MIC5504-1.8YM5, Y1 8MHz

Commit message: added journal entry
Parts:
- R15, R16, R17: footprint Package_DFN_QFN:WQFN-32-1EP_5x5mm_P0.5mm_EP3.1x3.1mm -> Resistor_SMD:R_0402_1005Metric
Changed lines of the file:
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@@
 			)
 		)
-		(property "Footprint" "Package_DFN_QFN:WQFN-32-1EP_5x5mm_P0.5mm_EP3.1x3.1mm"
+		(property "Footprint" "Resistor_SMD:R_0402_1005Metric"
 			(at 36.83 118.618 90)
 			(hide yes)
@@
 			)
 		)
-		(property "Footprint" "Package_DFN_QFN:WQFN-32-1EP_5x5mm_P0.5mm_EP3.1x3.1mm"
+		(property "Footprint" "Resistor_SMD:R_0402_1005Metric"
 			(at 36.83 133.858 90)
 			(hide yes)
@@
 			)
 		)
-		(property "Footprint" "Package_DFN_QFN:WQFN-32-1EP_5x5mm_P0.5mm_EP3.1x3.1mm"
+		(property "Footprint" "Resistor_SMD:R_0402_1005Metric"
 			(at 36.83 126.238 90)
 			(hide yes)

Commit message: set driver layout
Parts:
- removed D3, D4, D5, D6: BAT54C, Package_TO_SOT_SMD:SOT-23, symbol Diode:BAT54C
- added D10, D4, D6, D7: BAT54CW, Package_TO_SOT_SMD:SOT-323_SC-70, symbol Diode:BAT54CW
- C24, C25, C26, C27, C28, C29: footprint Capacitor_SMD:C_0402_1005Metric -> Capacitor_SMD:C_1210_3225Metric
Connections:
- net +3.3V: now also D10.3, D4.3, D6.3, D7.3
- net BEMF_A: now also D4.1
- net BEMF_B: now also D7.1
- net BEMF_C: now also D6.1
- net BEMF_U_A: now also D4.2
- net BEMF_U_B: now also D7.2
- net BEMF_U_C: now also D6.2
- net VGND: now also D10.1
- net at R15.2, R17.2: now also C21.1, R16.2, D10.2
- net at C19.1: now also U2.24 (DVDD); no longer U2.17 (DVDD)
- no-connect marks 0 -> 4
