File: bldc_driver.kicad_sch (KiCad schematic)
At the start: 58 parts, among them J1 Conn_01x01, J2 Conn_01x01, J3 Conn_01x01, Q1 DI030N10PT-AQ, Q2 DI030N10PT-AQ, Q3 DI030N10PT-AQ, Q4 DI030N10PT-AQ, Q5 DI030N10PT-AQ, Q6 DI030N10PT-AQ, Q7 Q_PMOS_DGS, U1 STM32F318K8Ux, U2 DRV8320SR, U4 MIC5504-1.8YM5, Y1 8MHz

Commit message: made next driver layout
Connections:
- net +3.3V: now also U4.3 (EN)
- net BEMF_A: no longer R11.2, R12.1, R13.2, R14.1
- net BEMF_B: now also R11.2, R12.1
- net BEMF_C: now also R13.2, R14.1
Other:
- moved on the sheet: C14, U4
Changed lines of the file:
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@@
 	)
 	(junction
-		(at 54.61 25.4)
+		(at 55.88 25.4)
 		(diameter 0)
 		(color 0 0 0 0)
@@
 	)
 	(junction
+		(at 30.48 25.4)
+		(diameter 0)
+		(color 0 0 0 0)
+	)
+	(junction
 		(at 246.38 35.56)
 		(diameter 0)
@@
 	(wire
 		(pts
+			(xy 31.75 30.48) (xy 30.48 30.48)
+		)
+		(stroke
+			(width 0)
+			(type default)
+		)
+	)
+	(wire
+		(pts
 			(xy 240.03 25.4) (xy 252.73 25.4)
 		)
@@
 	(wire
 		(pts
-			(xy 54.61 25.4) (xy 50.8 25.4)
+			(xy 55.88 25.4) (xy 52.07 25.4)
 		)
 		(stroke
@@
 	(wire
 		(pts
-			(xy 40.64 36.83) (xy 40.64 35.56)
+			(xy 41.91 36.83) (xy 41.91 35.56)
 		)
 		(stroke
@@
 	(wire
 		(pts
+			(xy 55.88 24.13) (xy 54.61 24.13)
+		)
+		(stroke
+			(width 0)
+			(type default)
+		)
+	)
+	(wire
+		(pts
 			(xy 252.73 99.06) (xy 260.35 99.06)
 		)
@@
 	(wire
 		(pts
+			(xy 30.48 25.4) (xy 30.48 30.48)
+		)
+		(stroke
+			(width 0)
+			(type default)
+		)
+	)
+	(wire
+		(pts
 			(xy 22.86 124.46) (xy 33.02 124.46)
 		)
@@
 	(wire
 		(pts
-			(xy 54.61 26.67) (xy 54.61 25.4)
+			(xy 55.88 26.67) (xy 55.88 25.4)
 		)
 		(stroke
@@
 	(wire
 		(pts
-			(xy 54.61 24.13) (xy 54.61 25.4)
+			(xy 55.88 24.13) (xy 55.88 25.4)
 		)
 		(stroke
@@
 	(wire
 		(pts
+			(xy 30.48 25.4) (xy 31.75 25.4)
+		)
+		(stroke
+			(width 0)
+			(type default)
+		)
+	)
+	(wire
+		(pts
 			(xy 129.54 74.93) (xy 149.86 74.93)
 		)
@@
 	(wire
 		(pts
-			(xy 54.61 35.56) (xy 54.61 34.29)
+			(xy 55.88 35.56) (xy 55.88 34.29)
 		)
 		(stroke
@@
 		)
 	)
-	(label "BEMF_A"
+	(label "BEMF_B"
 		(at 104.14 172.72 180)
 		(effects
@@
 		)
 	)
-	(label "BEMF_A"
+	(label "BEMF_C"
 		(at 153.67 172.72 180)
 		(effects
@@
 	)
 	(label "+1.8V"
-		(at 54.61 24.13 0)
+		(at 55.88 24.13 0)
 		(effects
 			(font
@@
 	(symbol
 		(lib_id "power:GND")
-		(at 40.64 36.83 0)
+		(at 41.91 36.83 0)
 		(unit 1)
 		(body_style 1)
@@
 		(dnp no)
 		(property "Reference" "#PWR026"
-			(at 40.64 43.18 0)
+			(at 41.91 43.18 0)
 			(hide yes)
 			(show_name no)
@@
 		)
 		(property "Value" "GND"
-			(at 40.64 40.894 0)
+			(at 41.91 40.894 0)
 			(show_name no)
 			(do_not_autoplace no)
@@
 		)
 		(property "Footprint" ""
-			(at 40.64 36.83 0)
+			(at 41.91 36.83 0)
 			(hide yes)
 			(show_name no)
@@
 		)
 		(property "Datasheet" ""
-			(at 40.64 36.83 0)
+			(at 41.91 36.83 0)
 			(hide yes)
 			(show_name no)
@@
 		)
 		(property "Description" "Power symbol creates a global label with name \"GND\" , ground"
-			(at 40.64 36.83 0)
+			(at 41.91 36.83 0)
 			(hide yes)
 			(show_name no)
@@
 	(symbol
 		(lib_id "power:GND")
-		(at 54.61 35.56 0)
+		(at 55.88 35.56 0)
 		(unit 1)
 		(body_style 1)
@@
 		(dnp no)
 		(property "Reference" "#PWR027"
-			(at 54.61 41.91 0)
+			(at 55.88 41.91 0)
 			(hide yes)
 			(show_name no)
@@
 		)
 		(property "Value" "GND"
-			(at 54.61 39.624 0)
+			(at 55.88 39.624 0)
 			(show_name no)
 			(do_not_autoplace no)
@@
 		)
 		(property "Footprint" ""
-			(at 54.61 35.56 0)
+			(at 55.88 35.56 0)
 			(hide yes)
 			(show_name no)
@@
 		)
 		(property "Datasheet" ""
-			(at 54.61 35.56 0)
+			(at 55.88 35.56 0)
 			(hide yes)
 			(show_name no)
@@
 		)
 		(property "Description" "Power symbol creates a global label with name \"GND\" , ground"
-			(at 54.61 35.56 0)
+			(at 55.88 35.56 0)
 			(hide yes)
 			(show_name no)
@@
 	(symbol
 		(lib_id "Regulator_Linear:MIC5504-1.8YM5")
-		(at 40.64 27.94 0)
+		(at 41.91 27.94 0)
 		(unit 1)
 		(body_style 1)
@@
 		(fields_autoplaced yes)
 		(property "Reference" "U4"
-			(at 40.64 17.78 0)
+			(at 41.91 17.78 0)
 			(show_name no)
 			(do_not_autoplace no)
@@
 		)
 		(property "Value" "MIC5504-1.8YM5"
-			(at 40.64 20.32 0)
+			(at 41.91 20.32 0)
 			(show_name no)
 			(do_not_autoplace no)
@@
 		)
 		(property "Footprint" "Package_TO_SOT_SMD:SOT-23-5"
-			(at 40.64 38.1 0)
+			(at 41.91 38.1 0)
 			(hide yes)
 			(show_name no)
@@
 		)
 		(property "Datasheet" "http://ww1.microchip.com/downloads/en/DeviceDoc/MIC550X.pdf"
-			(at 34.29 21.59 0)
+			(at 35.56 21.59 0)
 			(hide yes)
 			(show_name no)
@@
 		)
 		(property "Description" "300mA Low-dropout Voltage Regulator, Vout 1.8V, Vin up to 5.5V, SOT-23"
-			(at 40.64 27.94 0)
+			(at 41.91 27.94 0)
 			(hide yes)
 			(show_name no)
@@
 		)
 		(property "MPN" ""
-			(at 40.64 27.94 0)
+			(at 41.91 27.94 0)
 			(hide yes)
 			(show_name no)
@@
 	(symbol
 		(lib_id "Device:C")
-		(at 54.61 30.48 0)
+		(at 55.88 30.48 0)
 		(unit 1)
 		(body_style 1)
@@
 		(dnp no)
 		(property "Reference" "C14"
-			(at 55.88 28.194 0)
+			(at 57.15 28.194 0)
 			(show_name no)
 			(do_not_autoplace no)
@@
 		)
 		(property "Value" "1uF"
-			(at 55.88 33.274 0)
+			(at 57.15 33.274 0)
 			(show_name no)
 			(do_not_autoplace no)
@@
 		)
 		(property "Footprint" "Capacitor_SMD:C_0402_1005Metric"
-			(at 55.5752 34.29 0)
+			(at 56.8452 34.29 0)
 			(hide yes)
 			(show_name no)
@@
 		)
 		(property "Datasheet" ""
-			(at 54.61 30.48 0)
+			(at 55.88 30.48 0)
 			(hide yes)
 			(show_name no)
@@
 		)
 		(property "Description" "Unpolarized capacitor"
-			(at 54.61 30.48 0)
+			(at 55.88 30.48 0)
 			(hide yes)
 			(show_name no)
@@
 		)
 		(property "MPN" ""
-			(at 54.61 30.48 0)
+			(at 55.88 30.48 0)
 			(hide yes)
 			(show_name no)

Commit message: routing driver
Connections:
- net BEMF_A: no longer R10.1, R9.2
- net BEMF_B: no longer R11.2, R12.1
- net BEMF_C: no longer R13.2, R14.1
- net BEMF_U_A: now also R10.1, R9.2
- net BEMF_U_B: now also R11.2, R12.1
- net BEMF_U_C: now also R13.2, R14.1
- net DRV_EN: now also U1.23 (PA13)
- net FAULT: now also U1.29 (PB6)
- no-connect marks 4 -> 2
Changed lines of the file:
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@@
-	)
-	(no_connect
-		(at 129.54 85.09)
-	)
-	(no_connect
-		(at 99.06 82.55)
 	)
 	(no_connect
@@
 	(wire
 		(pts
+			(xy 129.54 85.09) (xy 139.7 85.09)
+		)
+		(stroke
+			(width 0)
+			(type default)
+		)
+	)
+	(wire
+		(pts
 			(xy 88.9 67.31) (xy 99.06 67.31)
 		)
@@
 	(wire
 		(pts
-			(xy 153.67 172.72) (xy 144.78 172.72)
+			(xy 156.21 172.72) (xy 144.78 172.72)
 		)
 		(stroke
@@
 	(wire
 		(pts
+			(xy 88.9 82.55) (xy 99.06 82.55)
+		)
+		(stroke
+			(width 0)
+			(type default)
+		)
+	)
+	(wire
+		(pts
 			(xy 96.52 25.4) (xy 88.9 25.4)
 		)
@@
 	(wire
 		(pts
-			(xy 104.14 172.72) (xy 95.25 172.72)
+			(xy 106.68 172.72) (xy 95.25 172.72)
 		)
 		(stroke
@@
 	(wire
 		(pts
-			(xy 54.61 172.72) (xy 45.72 172.72)
+			(xy 57.15 172.72) (xy 45.72 172.72)
 		)
 		(stroke
@@
 		)
 	)
-	(label "BEMF_B"
-		(at 104.14 172.72 180)
+	(label "BEMF_U_B"
+		(at 106.68 172.72 180)
 		(effects
 			(font
@@
 		)
 	)
-	(label "BEMF_C"
-		(at 153.67 172.72 180)
+	(label "BEMF_U_C"
+		(at 156.21 172.72 180)
 		(effects
 			(font
@@
 		)
 	)
+	(label "DRV_EN"
+		(at 139.7 85.09 180)
+		(effects
+			(font
+				(size 1.27 1.27)
+			)
+			(justify right bottom)
+		)
+	)
 	(label "IN_PWM"
 		(at 139.7 64.77 180)
@@
 		)
 	)
+	(label "FAULT"
+		(at 88.9 82.55 0)
+		(effects
+			(font
+				(size 1.27 1.27)
+			)
+			(justify left bottom)
+		)
+	)
 	(label "INHB"
 		(at 139.7 74.93 180)
@@
 		)
 	)
-	(label "BEMF_A"
-		(at 54.61 172.72 180)
-		(effects
-			(font
+	(label "BEMF_U_A"
+		(at 57.15 172.72 180)
+		(effects
+			(font

Commit message: routed driver
Connections:
- net SHB: now also U2.11 (SHB); no longer U2.9 (SLB)
Changed lines of the file:
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@@
 		(pin "8"
 		)
-		(pin "9"
+		(pin "11"
 		)
 		(pin "9"
