File: Multi-ESC.kicad_pcb (KiCad board)
At the start: 4 copper layers, 252 parts, among them J1 Conn_01x01, J10 Conn_01x01, J11 Conn_01x01, J12 Conn_01x01, J13 Conn_01x01, J14 Conn_01x01, J15 Conn_01x01, J16 Conn_01x01, J17 Conn_01x03, J18 Conn_01x05, J2 Conn_01x01, J3 Conn_01x01, J4 Conn_01x01, J5 Conn_01x01, J6 Conn_01x01, J7 Conn_01x01, J8 Conn_01x01, J9 Conn_01x01, Q1 DI030N10PT-AQ, Q10 DI030N10PT-AQ, Q11 DI030N10PT-AQ, Q12 DI030N10PT-AQ, Q13 DI030N10PT-AQ, Q14 Q_PMOS_DGS, Q15 DI030N10PT-AQ, Q16 DI030N10PT-AQ, Q17 DI030N10PT-AQ, Q18 DI030N10PT-AQ, Q19 DI030N10PT-AQ, Q2 DI030N10PT-AQ, Q20 DI030N10PT-AQ, Q21 Q_PMOS_DGS, Q22 DI030N10PT-AQ, Q23 DI030N10PT-AQ, Q24 DI030N10PT-AQ, Q25 DI030N10PT-AQ, Q26 DI030N10PT-AQ, Q27 DI030N10PT-AQ, Q28 Q_PMOS_DGS, Q3 DI030N10PT-AQ, Q4 DI030N10PT-AQ, Q5 DI030N10PT-AQ, Q6 DI030N10PT-AQ, Q7 Q_PMOS_DGS, Q8 DI030N10PT-AQ, Q9 DI030N10PT-AQ, U1 STM32F318K8Ux, U10 DRV8320SR, U11 MIC5504-1.8YM5, U12 STM32F318K8Ux, U13 DRV8320SR, U2 DRV8320SR, U3 LMR51450FN, U4 MIC5504-1.8YM5, U5 MIC5504-1.8YM5, U6 STM32F318K8Ux, U7 DRV8320SR, U8 MIC5504-1.8YM5, U9 STM32F318K8Ux, Y1 8MHz, Y2 8MHz, Y3 8MHz, Y4 8MHz

Commit message: routed driver
Connections:
- U10 pad 11: (no net) -> /BLDC Driver2/SHB
- U10 pad 9: /BLDC Driver2/SHB -> GND
- U13 pad 11: (no net) -> /BLDC Driver3/SHB
- U13 pad 9: /BLDC Driver3/SHB -> GND
- U2 pad 11: (no net) -> /BLDC Driver0/SHB
- U2 pad 9: /BLDC Driver0/SHB -> GND
- U7 pad 11: (no net) -> /BLDC Driver1/SHB
- U7 pad 9: /BLDC Driver1/SHB -> GND
Routing:
- net /BLDC Driver0/+1.8V: track 6.74 -> 42.3 mm, vias 1 -> 6
- net GND: track 0.00 -> 29.2 mm, vias 0 -> 9
- net /BLDC Driver0/BEMF_U_A: track 7.96 -> 36.6 mm, vias 2 -> 3
- net /BLDC Driver0/BEMF_U_B: track 11.2 -> 34.8 mm, vias 2 -> 3
- net /BLDC Driver0/BEMF_U_C: track 12.6 -> 34.9 mm, vias 2 -> 3
- net /BLDC Driver0/GHA: track 0.00 -> 20.7 mm, vias 0 -> 2
- net /BLDC Driver0/GLA: track 0.00 -> 20.7 mm, vias 0 -> 2
- net /BLDC Driver0/SHA: track 0.00 -> 19.4 mm, vias 0 -> 2
- net /BLDC Driver0/SHC: track 0.00 -> 18.3 mm, vias 0 -> 2
- net +3.3V: track 7.82 -> 23.1 mm, vias 0 -> 3
- net /BLDC Driver0/SHB: track 0.00 -> 13.5 mm, vias 0 -> 2
- net /BLDC Driver0/GLC: track 0.00 -> 12.9 mm, vias 0 -> 2
- net /BLDC Driver0/GHC: track 0.00 -> 12.2 mm, vias 0 -> 2
- net /BLDC Driver0/GLB: track 0.00 -> 12.2 mm, vias 0 -> 2
- net /BLDC Driver0/GHB: track 0.00 -> 10.6 mm, vias 0 -> 2
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- added copper zone on F.Cu, net /BLDC Driver0/SHA
- added copper zone on F.Cu, net /BLDC Driver0/SHB
- added copper zone on F.Cu, net /BLDC Driver0/SHC
- added copper zone on F.Cu, net /BLDC Driver0/VM

Commit message: made rest of driver layout
Parts:
- moved D19 321.9 mm to (136.1, 135.4), turned to -90 degrees
- moved J12 318.0 mm to (167.6, 122.0)
- moved J13 317.6 mm to (167.6, 129.0)
- moved J14 317.2 mm to (167.6, 136.0)
- moved D14 308.2 mm to (143.3, 135.4), turned to -90 degrees
- moved D17 304.8 mm to (140.9, 135.4), turned to -90 degrees
- moved D25 301.3 mm to (138.5, 135.4), turned to -90 degrees
- moved R44 297.6 mm to (133.9, 133.6)
- moved R51 292.4 mm to (162.9, 138.0), turned to 180 degrees
- moved R52 292.2 mm to (161.0, 138.0), turned to 180 degrees
- moved R45 292.1 mm to (133.9, 134.6)
- moved U13 291.6 mm to (149.5, 130.8), turned to 90 degrees
- moved R49 290.8 mm to (162.8, 131.0), turned to 180 degrees
- moved R47 289.4 mm to (162.8, 124.0), turned to 180 degrees
- moved U12 289.0 mm to (142.2, 129.9)
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