File: Multi-ESC.kicad_pcb (KiCad board)
At the start: 4 copper layers, 252 parts, among them J1 Conn_01x01, J10 Conn_01x01, J11 Conn_01x01, J12 Conn_01x01, J13 Conn_01x01, J14 Conn_01x01, J15 Conn_01x01, J16 Conn_01x01, J17 Conn_01x03, J18 Conn_01x05, J2 Conn_01x01, J3 Conn_01x01, J4 Conn_01x01, J5 Conn_01x01, J6 Conn_01x01, J7 Conn_01x01, J8 Conn_01x01, J9 Conn_01x01, Q1 DI030N10PT-AQ, Q10 DI030N10PT-AQ, Q11 DI030N10PT-AQ, Q12 DI030N10PT-AQ, Q13 DI030N10PT-AQ, Q14 Q_PMOS_DGS, Q15 DI030N10PT-AQ, Q16 DI030N10PT-AQ, Q17 DI030N10PT-AQ, Q18 DI030N10PT-AQ, Q19 DI030N10PT-AQ, Q2 DI030N10PT-AQ, Q20 DI030N10PT-AQ, Q21 Q_PMOS_DGS, Q22 DI030N10PT-AQ, Q23 DI030N10PT-AQ, Q24 DI030N10PT-AQ, Q25 DI030N10PT-AQ, Q26 DI030N10PT-AQ, Q27 DI030N10PT-AQ, Q28 Q_PMOS_DGS, Q3 DI030N10PT-AQ, Q4 DI030N10PT-AQ, Q5 DI030N10PT-AQ, Q6 DI030N10PT-AQ, Q7 Q_PMOS_DGS, Q8 DI030N10PT-AQ, Q9 DI030N10PT-AQ, U1 STM32F318K8Ux, U10 DRV8320SR, U11 MIC5504-1.8YM5, U12 STM32F318K8Ux, U13 DRV8320SR, U2 DRV8320SR, U3 LMR51450FN, U4 MIC5504-1.8YM5, U5 MIC5504-1.8YM5, U6 STM32F318K8Ux, U7 DRV8320SR, U8 MIC5504-1.8YM5, U9 STM32F318K8Ux, Y1 8MHz, Y2 8MHz, Y3 8MHz, Y4 8MHz

Commit message: added journal entry
Parts:
- moved C83 54.0 mm to (120.1, 78.6)
- moved Q24 54.0 mm to (141.9, 76.9)
- moved R44 54.0 mm to (118.3, 81.8)
- moved R46 54.0 mm to (118.3, 83.8)
- moved R45 54.0 mm to (118.3, 82.8)
- moved C75 54.0 mm to (114.9, 83.7)
- moved C78 54.0 mm to (124.3, 74.1)
- moved C79 54.0 mm to (129.3, 82.0)
- moved C80 54.0 mm to (123.3, 75.1)
- moved C81 54.0 mm to (122.2, 79.7)
- moved C82 54.0 mm to (122.2, 78.7)
- moved C84 54.0 mm to (120.7, 74.0)
- moved C85 54.0 mm to (133.2, 64.6)
- moved C86 54.0 mm to (122.3, 64.6)
- moved C87 54.0 mm to (130.4, 81.9)
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
Commit message: started routing
Parts:
- moved R43 0.13 mm to (66.0, 73.5)
Routing:
- net /BLDC Driver2/BEMF_U_C: track 0.00 -> 33.9 mm, vias 0 -> 2
- net /BLDC Driver2/SHA: track 0.00 -> 24.6 mm, vias 0 -> 1
- net /BLDC Driver2/GHA: track 0.00 -> 24.0 mm, vias 0 -> 2
- net /BLDC Driver2/GLA: track 0.00 -> 22.7 mm, vias 0 -> 2
- net /BLDC Driver2/SHC: track 0.00 -> 18.3 mm, vias 0 -> 1
- net /BLDC Driver2/SHB: track 0.00 -> 18.0 mm, vias 0 -> 1
- net /BLDC Driver2/CS: track 0.00 -> 16.9 mm, vias 0 -> 2
- net /BLDC Driver2/GLB: track 0.00 -> 12.9 mm, vias 0 -> 2
- net /BLDC Driver2/BEMF_U_B: track 0.00 -> 12.2 mm, vias 0 -> 3
- net /BLDC Driver2/GLC: track 0.00 -> 11.4 mm, vias 0 -> 2
- net /BLDC Driver2/GHB: track 0.00 -> 10.0 mm, vias 0 -> 2
- net /BLDC Driver2/INHC: track 0.00 -> 8.99 mm, vias 0 -> 2
- net /BLDC Driver2/GHC: track 0.00 -> 8.98 mm, vias 0 -> 2
- net /BLDC Driver2/INLC: track 0.00 -> 8.25 mm, vias 0 -> 2
- net /BLDC Driver2/BEMF_U_A: track 0.00 -> 8.25 mm, vias 0 -> 3
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
Commit message: routing drivers 2 and 3
Parts:
- added BOOT1: SW_Push, Button_Switch_SMD:SW_Push_SPST_NO_Alps_SKRK, F.Cu at (276.7, 131.8)
- added R57: 10K, Resistor_SMD:R_0402_1005Metric, F.Cu at (274.9, 135.0)
- moved C38 0.44 mm to (124.0, 41.4)
- moved C37 0.44 mm to (124.0, 42.4)
- moved C46 0.43 mm to (133.7, 45.5)
- moved C11 0.20 mm to (57.9, 39.7)
- moved C12 0.20 mm to (57.9, 38.7)
- turned R28 to -90 degrees
- turned R29 to -90 degrees
Connections:
- Q8 pad 2: /BLDC Driver1/GHA -> (no net)
Routing:
- net /BLDC Driver2/+1.8V: track 6.08 -> 42.7 mm, vias 0 -> 7
- net /BLDC Driver1/CS: track 0.00 -> 16.3 mm, vias 0 -> 2
- net /BLDC Driver1/FAULT: track 0.00 -> 16.1 mm
- net /BLDC Driver2/FAULT: track 1.46 -> 16.8 mm
- net GND: track 29.2 -> 44.4 mm, vias 9 -> 12
- net /BLDC Driver1/VM: track 0.00 -> 13.3 mm
- net /BLDC Driver2/MOSI: track 0.00 -> 12.0 mm
- net /BLDC Driver1/BEMF_U_C: track 0.00 -> 11.9 mm, vias 0 -> 2
- net /BLDC Driver1/MOSI: track 0.00 -> 11.7 mm
- net /BLDC Driver0/VM: track 3.58 -> 14.4 mm
- net /BLDC Driver1/MISO: track 0.00 -> 10.7 mm, vias 0 -> 2
- net /BLDC Driver2/VM: track 4.14 -> 14.4 mm
- net /BLDC Driver2/MISO: track 1.65 -> 11.7 mm, vias 0 -> 2
- net /BLDC Driver2/SCLK: track 0.00 -> 9.75 mm
- net /BLDC Driver1/BEMF_U_B: track 0.00 -> 9.73 mm, vias 0 -> 2
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- added copper zone on F.Cu, net /BLDC Driver2/SHA
- added copper zone on F.Cu, net /BLDC Driver2/SHB
- added copper zone on F.Cu, net /BLDC Driver2/SHC
- added copper zone on F.Cu, net /BLDC Driver2/VM

Commit message: edited footprints
Connections:
- Q10 pad 3: (no net) -> /BLDC Driver1/SHB
- Q11 pad 3: (no net) -> GND
- Q8 pad 2: (no net) -> /BLDC Driver1/GHA
- Q8 pad 3: /BLDC Driver1/GHA -> /BLDC Driver1/SHA
- Q9 pad 3: (no net) -> GND
Changed lines of the file:
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@@
 		(sheetname "/BLDC Driver1/")
 		(sheetfile "bldc_driver.kicad_sch")
+		(units
+			(unit
+				(name "A")
+				(pins "2" "1" "3")
+			)
+		)
 		(attr smd)
 		(duplicate_pad_numbers_are_jumpers no)
@@
 			(size 0.4 0.4)
 			(layers "F.Cu" "F.Mask" "F.Paste")
+			(net "/BLDC Driver1/SHB")
+			(pinfunction "S_3")
+			(pintype "passive")
 			(zone_connect 2)
 			(options
@@
 		(sheetname "/BLDC Driver1/")
 		(sheetfile "bldc_driver.kicad_sch")
+		(units
+			(unit
+				(name "A")
+				(pins "2" "1" "3")
+			)
+		)
 		(attr smd)
 		(duplicate_pad_numbers_are_jumpers no)
@@
 			(size 0.4 0.4)
 			(layers "F.Cu" "F.Mask" "F.Paste")
+			(net "GND")
+			(pinfunction "S_3")
+			(pintype "passive")
 			(zone_connect 2)
 			(options
@@
 		(sheetname "/BLDC Driver1/")
 		(sheetfile "bldc_driver.kicad_sch")
+		(units
+			(unit
+				(name "A")
+				(pins "2" "1" "3")
+			)
+		)
 		(attr smd)
 		(duplicate_pad_numbers_are_jumpers no)
@@
 			(size 0.4 0.4)
 			(layers "F.Cu" "F.Mask" "F.Paste")
+			(net "GND")
+			(pinfunction "S_3")
+			(pintype "passive")
 			(zone_connect 2)
 			(options
@@
 		(sheetname "/BLDC Driver1/")
 		(sheetfile "bldc_driver.kicad_sch")
+		(units
+			(unit
+				(name "A")
+				(pins "2" "1" "3")
+			)
+		)
 		(attr smd)
 		(duplicate_pad_numbers_are_jumpers no)
@@
 			(size 0.8 0.44)
 			(layers "F.Cu" "F.Mask" "F.Paste")
+			(net "/BLDC Driver1/GHA")
+			(pinfunction "G_2")
+			(pintype "input")
 		)
 		(pad "3" smd custom
@@
 			(size 0.4 0.4)
 			(layers "F.Cu" "F.Mask" "F.Paste")
-			(net "/BLDC Driver1/GHA")
-			(pinfunction "G_2")
-			(pintype "input")
+			(net "/BLDC Driver1/SHA")
+			(pinfunction "S_3")
+			(pintype "passive")
 			(zone_connect 2)
 			(options

Commit message: finished routing other drivers
Parts:
- moved C84 4.68 mm to (120.0, 78.6)
- moved C83 4.59 mm to (120.5, 74.0)
- moved C90 0.30 mm to (131.8, 83.0)
- moved C92 0.27 mm to (133.3, 83.1)
- moved C43 0.26 mm to (132.1, 44.2)
- moved C76 0.18 mm to (120.3, 81.7)
- turned R25 to 180 degrees
- turned Y4 to 180 degrees
Connections:
- U6 pad 12: /PWM0 -> /PWM1
- U9 pad 12: /PWM1 -> /PWM2
Routing:
- net +3.3V: track 33.0 -> 93.2 mm, vias 3 -> 15
- net GND: track 44.4 -> 100.4 mm, vias 12 -> 32
- net /BLDC Driver3/+1.8V: track 0.00 -> 40.0 mm, vias 0 -> 6
- net /BLDC Driver3/BEMF_U_A: track 0.00 -> 37.1 mm, vias 0 -> 3
- net /BLDC Driver1/+1.8V: track 4.58 -> 39.7 mm, vias 0 -> 6
- net /BLDC Driver3/BEMF_U_B: track 0.00 -> 33.9 mm, vias 0 -> 3
- net /BLDC Driver3/BEMF_U_C: track 0.00 -> 33.5 mm, vias 0 -> 2
- net /BLDC Driver1/BEMF_U_A: track 5.94 -> 35.4 mm, vias 2 -> 3
- net /BLDC Driver1/SHA: track 0.00 -> 26.8 mm, vias 0 -> 1
- net /BLDC Driver1/BEMF_U_B: track 9.73 -> 34.5 mm, vias 2 -> 3
- net /BLDC Driver3/SHA: track 0.00 -> 24.1 mm, vias 0 -> 1
- net /BLDC Driver3/GHA: track 0.00 -> 23.6 mm, vias 0 -> 2
- net /BLDC Driver1/GHA: track 0.00 -> 23.0 mm, vias 0 -> 2
- net /BLDC Driver3/GLA: track 0.00 -> 22.0 mm, vias 0 -> 2
- net /BLDC Driver1/BEMF_U_C: track 11.9 -> 33.7 mm
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- added copper zone on F.Cu, net /BLDC Driver1/SHA
- added copper zone on F.Cu, net /BLDC Driver1/SHB
- added copper zone on F.Cu, net /BLDC Driver1/SHC
- added copper zone on F.Cu, net /BLDC Driver1/VM
- added copper zone on F.Cu, net /BLDC Driver3/SHA
- added copper zone on F.Cu, net /BLDC Driver3/SHB
- added copper zone on F.Cu, net /BLDC Driver3/SHC
- added copper zone on F.Cu, net /BLDC Driver3/VM

Commit message: started routing whole board
Parts:
- TP1, TP10, TP11, TP12, TP13, TP14, TP15, TP16, TP2, TP3, TP4, TP5, TP6, TP7, TP8, TP9: moved to B.Cu
- moved D2 148.9 mm to (136.8, 67.0), turned to 180 degrees
- moved J4 147.7 mm to (133.3, 61.5), turned to -90 degrees
- moved C7 147.4 mm to (134.3, 94.8), turned to 180 degrees
- moved C6 146.1 mm to (134.3, 93.2), turned to 180 degrees
- moved J5 145.9 mm to (140.3, 61.5), turned to -90 degrees
- moved C5 144.9 mm to (134.3, 91.6), turned to 180 degrees
- moved R2 144.8 mm to (132.9, 89.2), turned to 180 degrees
- moved R1 144.1 mm to (132.9, 88.2), turned to 0 degrees
- moved C4 143.2 mm to (134.9, 90.2), turned to 180 degrees
- moved R3 142.3 mm to (133.2, 86.2), turned to -90 degrees
- moved U3 140.2 mm to (135.7, 87.4), turned to -90 degrees
- moved R4 139.4 mm to (134.4, 84.2), turned to 90 degrees
- moved BOOT1 138.3 mm to (140.8, 106.3)
- moved C1 137.7 mm to (136.0, 84.6), turned to 0 degrees
- moved R57 136.7 mm to (140.7, 108.6), turned to 180 degrees
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Routing:
- net /BLDC Driver2/BEMF_U_A: track 8.25 -> 37.0 mm
- net +3.3V: track 93.2 -> 114.4 mm
- net /BLDC Driver3/NPOR: track 0.00 -> 14.6 mm, vias 0 -> 2
- net /BLDC Driver0/NPOR: track 1.42 -> 15.9 mm, vias 1 -> 2
- net Net-(C1-Pad2): track 0.00 -> 13.8 mm
- net /BLDC Driver1/NPOR: track 1.05 -> 14.7 mm, vias 1 -> 2
- net /BLDC Driver2/NPOR: track 1.21 -> 14.7 mm, vias 1 -> 2
- net /BLDC Driver2/NRST: track 0.91 -> 11.8 mm, vias 1 -> 2
- net /BLDC Driver1/NRST: track 0.99 -> 11.9 mm, vias 1 -> 2
- net /BLDC Driver0/NRST: track 1.20 -> 11.9 mm, vias 1 -> 2
- net /BLDC Driver0/INLA: track 2.73 -> 13.3 mm, vias 0 -> 1
- net /BLDC Driver3/NRST: track 0.95 -> 11.2 mm, vias 1 -> 2
- net /BLDC Driver1/INLA: track 2.60 -> 12.7 mm, vias 0 -> 1
- net /BLDC Driver3/INLA: track 2.70 -> 12.7 mm, vias 0 -> 1
- net /BLDC Driver2/INLA: track 2.67 -> 12.5 mm, vias 0 -> 1
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Other:
- board outline added: 110 x 70 mm
- board text added: "BOOT"
- board text added: "NPOR"
- board text added: "NRST"
- board text added: "RX"
- board text added: "TX"
