File: Multi-ESC.kicad_sch (KiCad schematic)
At the start: 21 parts, among them J15 Conn_01x01, J16 Conn_01x01, J17 Conn_01x03, J18 Conn_01x05, J4 Conn_01x01, J5 Conn_01x01, U3 LMR51450FN

Commit message: routing drivers 2 and 3
Parts:
- added BOOT1: SW_Push, Button_Switch_SMD:SW_Push_SPST_NO_Alps_SKRK, symbol Switch:SW_Push
- added R57: 10K, Resistor_SMD:R_0402_1005Metric, symbol Device:R
Connections:
- net +3.3V: now also BOOT1.1
- net BOOT: now also BOOT1.2, R57.1
- net GND: now also R57.2

Commit message: finished routing other drivers
Changed lines of the file:
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@@
 		)
 	)
-	(label "PWM0"
+	(label "PWM1"
 		(at 19.05 49.53 0)
 		(effects
@@
 		)
 	)
-	(label "PWM1"
+	(label "PWM2"
 		(at 19.05 71.12 0)
 		(effects
